Commit message: added gazebo launch file

File: milo_ws/src/milo_description/models/milo_bot/robot_core.xacro (robot description, xacro)
@@ -29,5 +29,5 @@
         <parent link="base_link"/>
         <child link="chassis_link"/>
-        <origin xyz="0 0 0"/>
+        <origin xyz="0 0 0.035"/>
     </joint>
     <link name="chassis_link">
@@ -49,9 +49,12 @@
         </xacro:inertial_box>
     </link>
+    <gazebo reference="chassis_link">
+        <material>Gazebo/White</material>
+    </gazebo>
     <!-- LEFT REAR WHEEL LINK -->
     <joint name="left_rear_wheel_joint" type="continuous">
         <parent link="base_link"/>
         <child link="left_rear_wheel_link"/>
-        <origin xyz="-0.05 0.125 0" rpy="-${pi/2} 0 0"/>
+        <origin xyz="-0.05 0.125 0.035" rpy="-${pi/2} 0 0"/>
         <axis xyz="0 0 1"/>
     </joint>
@@ -75,9 +78,12 @@
         </xacro:inertial_cylinder>
     </link>
+    <gazebo reference="left_rear_wheel_link">
+        <material>Gazebo/Orange</material>
+    </gazebo>
     <!-- LEFT FRONT WHEEL LINK -->
     <joint name="left_front_wheel_joint" type="continuous">
         <parent link="base_link"/>
         <child link="left_front_wheel_link"/>
-        <origin xyz="0.05 0.125 0" rpy="-${pi/2} 0 0"/>
+        <origin xyz="0.05 0.125 0.035" rpy="-${pi/2} 0 0"/>
         <axis xyz="0 0 1"/>
     </joint>
@@ -101,9 +107,12 @@
         </xacro:inertial_cylinder>
     </link>
+    <gazebo reference="left_front_wheel_link">
+        <material>Gazebo/Orange</material>
+    </gazebo>
     <!-- RIGHT REAR WHEEL LINK -->
     <joint name="right_rear_wheel_joint" type="continuous">
         <parent link="base_link"/>
         <child link="right_rear_wheel_link"/>
-        <origin xyz="-0.05 -0.125 0" rpy="${pi/2} 0 0"/>
+        <origin xyz="-0.05 -0.125 0.035" rpy="${pi/2} 0 0"/>
         <axis xyz="0 0 1"/>
     </joint>
@@ -127,9 +136,12 @@
         </xacro:inertial_cylinder>
     </link>
+    <gazebo reference="right_rear_wheel_link">
+        <material>Gazebo/Orange</material>
+    </gazebo>
     <!-- RIGHT FRONT WHEEL LINK -->
     <joint name="right_front_wheel_joint" type="continuous">
         <parent link="base_link"/>
         <child link="right_front_wheel_link"/>
-        <origin xyz="0.05 -0.125 0" rpy="${pi/2} 0 0"/>
+        <origin xyz="0.05 -0.125 0.035" rpy="${pi/2} 0 0"/>
         <axis xyz="0 0 1"/>
     </joint>
@@ -153,9 +165,12 @@
         </xacro:inertial_cylinder>
     </link>
+    <gazebo reference="right_front_wheel_link">
+        <material>Gazebo/Orange</material>
+    </gazebo>
     <!-- CAMERA STAND LINK -->
     <joint name="camera_stand_joint" type="fixed">
         <parent link="base_link"/>
         <child link="camera_stand_link"/>
-        <origin xyz="0.105 0 0.125" rpy="0 ${pi/2} 0"/>
+        <origin xyz="0.105 0 0.160" rpy="0 ${pi/2} 0"/>
     </joint>
     <link name="camera_stand_link">
@@ -178,3 +193,6 @@
         </xacro:inertial_box>
     </link>
+    <gazebo reference="camera_stand_link">
+        <material>Gazebo/White</material>
+    </gazebo>
 </robot>
