Commit message: minimal working version of diff_drive bot in gazebo

File: milo_ws/src/milo_description/models/milo_bot/gazebo_control.xacro (robot description, xacro)
@@ -2,20 +2,36 @@
 <robot xmlns:xacro="https://www.ros.org/wiki/xacro" name="robot">
     <gazebo>
-        <plugin name="diff_drive" filename="libgazebo_ros_diff_drive.so">
-        <!-- Wheel information -->
-        <left_joint>left_rear_wheel_joint</left_joint>
-        <right_joint>right_rear_wheel_joint</right_joint>
-        <wheel_separation>0.250</wheel_separation>
-        <wheel_diameter>0.070</wheel_diameter>
-        <!-- Limits -->
-        <max_wheel_torque>200</max_wheel_torque>
-        <max_wheel_acceleration>10.0</max_wheel_acceleration>
-        <!-- Output -->
-        <odometry_frame>odom</odometry_frame>
-        <robot_base_frame>base_link</robot_base_frame>
-        <publish_odom>true</publish_odom>
-        <publish_odom_tf>true</publish_odom_tf>
-        <publish_wheel_transform>true</publish_wheel_transform>
+        <plugin name='diff_drive' filename='libgazebo_ros_diff_drive.so'>
+            <!-- Wheel Information -->
+            <left_joint>left_rear_wheel_joint</left_joint>
+            <right_joint>right_rear_wheel_joint</right_joint>
+            <wheel_separation>0.35</wheel_separation>
+            <wheel_diameter>0.1</wheel_diameter>
+            <!-- Limits -->
+            <max_wheel_torque>200</max_wheel_torque>
+            <max_wheel_acceleration>10.0</max_wheel_acceleration>
+            <!-- Output -->
+            <odometry_frame>odom</odometry_frame>
+            <robot_base_frame>base_link</robot_base_frame>
+            <publish_odom>true</publish_odom>
+            <publish_odom_tf>true</publish_odom_tf>
+            <publish_wheel_tf>true</publish_wheel_tf>
         </plugin>
     </gazebo>
+<!-- <gazebo>
+  <plugin name="skid_steer_drive_controller" filename="libgazebo_ros_skid_steer_drive.so">
+    <updateRate>100.0</updateRate>
+    <robotNamespace>/</robotNamespace>
+    <leftFrontJoint>front_left_wheel_joint</leftFrontJoint>
+    <rightFrontJoint>front_right_wheel_joint</rightFrontJoint>
+    <leftRearJoint>back_left_wheel_joint</leftRearJoint>
+    <rightRearJoint>back_right_wheel_joint</rightRearJoint>
+    <wheelSeparation>0.4</wheelSeparation>
+    <wheelDiameter>0.215</wheelDiameter>
+    <robotBaseFrame>base_link</robotBaseFrame>
+    <torque>20</torque>
+    <topicName>cmd_vel</topicName>
+    <broadcastTF>true</broadcastTF>
+  </plugin>
+</gazebo> -->
 </robot>

File: milo_ws/src/milo_description/models/milo_bot/robot_core.xacro (robot description, xacro)
@@ -1,37 +1,28 @@
 <?xml version="1.0"?>
-<robot xmlns:xacro="https://www.ros.org/wiki/xacro" name="robot">
-    <!-- Include inertial macros -->
-    <xacro:include filename="inertial_macros.xacro"/>
-    <!-- Set up colours -->
+<robot xmlns:xacro="http://www.ros.org/wiki/xacro">
+<xacro:include filename="inertial_macros.xacro" />
     <material name="white">
-        <color rgba="1 1 1 1" />
+        <color rgba="1 1 1 1"/>
     </material>
     <material name="orange">
-        <color rgba="1 0.3 0.1 1" />
-    </material>
-    <material name="red">
-        <color rgba="1 0 0 1" />
-    </material>
-    <material name="green">
-        <color rgba="0 1 0 1" />
+        <color rgba="1 0.3 0.1 1"/>
     </material>
     <material name="blue">
-        <color rgba="0 0 1 1" />
+        <color rgba="0.2 0.2 1 1"/>
     </material>
     <material name="black">
-        <color rgba="0 0 0 1" />
+        <color rgba="0 0 0 1"/>
     </material>
-    <!-- BASE LINK -->
     <link name="base_link">
     </link>
-    <!-- CHASSIS LINK -->
+    <!-- CHASSIS -->
     <joint name="chassis_joint" type="fixed">
         <parent link="base_link"/>
-        <child link="chassis_link"/>
-        <origin xyz="0 0 0.035"/>
+        <child link="chassis"/>
+        <origin xyz="0 0 0.0525"/>
     </joint>
-    <link name="chassis_link">
+    <link name="chassis">
         <visual>
-            <origin xyz="0 0 0.0525" rpy="0 0 0"/>
+            <origin xyz="0 0 0" rpy="0 0 0"/>
             <geometry>
                 <box size="0.220 0.210 0.105"/>
@@ -40,163 +31,67 @@
         </visual>
         <collision>
-            <origin xyz="0 0 0.0525"/>
+            <origin xyz="0 0 0" rpy="0 0 0"/>
             <geometry>
                 <box size="0.220 0.210 0.105"/>
             </geometry>
         </collision>
-        <xacro:inertial_box mass="0.5" x="0.220" y="0.210" z="0.105">
-            <origin xyz="0 0 0.0525" rpy="0 0 0"/>
+        <xacro:inertial_box mass="0.1" x="0.220" y="0.210" z="0.105">
+            <origin xyz="0 0 0" rpy="0 0 0"/>
         </xacro:inertial_box>
     </link>
-    <gazebo reference="chassis_link">
+    <gazebo reference="chassis">
         <material>Gazebo/White</material>
     </gazebo>
-    <!-- LEFT REAR WHEEL LINK -->
+    <!-- LEFT REAR WHEEL -->
     <joint name="left_rear_wheel_joint" type="continuous">
         <parent link="base_link"/>
-        <child link="left_rear_wheel_link"/>
-        <origin xyz="-0.05 0.125 0.035" rpy="-${pi/2} 0 0"/>
+        <child link="left_rear_wheel"/>
+        <origin xyz="-0.05 0.1125 0" rpy="-${pi/2} 0 0"/>
         <axis xyz="0 0 1"/>
     </joint>
-    <link name="left_rear_wheel_link">
+    <link name="left_rear_wheel">
         <visual>
-            <origin xyz="0 0 0"/>
             <geometry>
-                <cylinder radius="0.035" length="0.04"/>
+                <cylinder length="0.025" radius="0.035" />
             </geometry>
-            <material name="orange"/>
+            <material name="blue"/>
         </visual>
         <collision>
-            <origin xyz="0 0 0"/>
             <geometry>
-                <cylinder radius="0.035" length="0.04"/>
+                <cylinder length="0.025" radius="0.035" />
             </geometry>
-            <material name="orange"/>
         </collision>
-        <xacro:inertial_cylinder mass="0.1" length="0.04" radius="0.035">
+        <xacro:inertial_cylinder mass="0.1" length="0.025" radius="0.035">
             <origin xyz="0 0 0" rpy="0 0 0"/>
         </xacro:inertial_cylinder>
     </link>
-    <gazebo reference="left_rear_wheel_link">
-        <material>Gazebo/Orange</material>
+    <gazebo reference="left_rear_wheel">
+        <material>Gazebo/Red</material>
     </gazebo>
-    <!-- LEFT FRONT WHEEL LINK -->
-    <joint name="left_front_wheel_joint" type="continuous">
+    <!-- RIGHT WHEEL -->
+    <joint name="right_rear_wheel_joint" type="continuous">
         <parent link="base_link"/>
-        <child link="left_front_wheel_link"/>
-        <origin xyz="0.05 0.125 0.035" rpy="-${pi/2} 0 0"/>
-        <axis xyz="0 0 1"/>
+        <child link="right_rear_wheel"/>
+        <origin xyz="-0.050 -0.1125 0" rpy="${pi/2} 0 0"/>
+        <axis xyz="0 0 -1"/>
     </joint>
-    <link name="left_front_wheel_link">
+    <link name="right_rear_wheel">
         <visual>
-            <origin xyz="0 0 0"/>
             <geometry>
-                <cylinder radius="0.035" length="0.04"/>
+                <cylinder length="0.025" radius="0.035" />
             </geometry>
-            <material name="orange"/>
+            <material name="blue"/>
         </visual>
         <collision>
-            <origin xyz="0 0 0"/>
             <geometry>
-                <cylinder radius="0.035" length="0.04"/>
+                <cylinder length="0.025" radius="0.035" />
             </geometry>
-            <material name="orange"/>
         </collision>
-        <xacro:inertial_cylinder mass="0.1" length="0.04" radius="0.035">
+        <xacro:inertial_cylinder mass="0.1" length="0.025" radius="0.035">
             <origin xyz="0 0 0" rpy="0 0 0"/>
         </xacro:inertial_cylinder>
     </link>
-    <gazebo reference="left_front_wheel_link">
-        <material>Gazebo/Orange</material>
-        <mu1 value="0.5"/>
-        <mu2 value="0.5"/>
-    </gazebo>
-    <!-- RIGHT REAR WHEEL LINK -->
-    <joint name="right_rear_wheel_joint" type="continuous">
-        <parent link="base_link"/>
-        <child link="right_rear_wheel_link"/>
-        <origin xyz="-0.05 -0.125 0.035" rpy="${pi/2} 0 0"/>
-        <axis xyz="0 0 1"/>
-    </joint>
-    <link name="right_rear_wheel_link">
-        <visual>
-            <origin xyz="0 0 0"/>
-            <geometry>
-                <cylinder radius="0.035" length="0.04"/>
-            </geometry>
-            <material name="orange"/>
-        </visual>
-        <collision>
-            <origin xyz="0 0 0"/>
-            <geometry>
-                <cylinder radius="0.035" length="0.04"/>
-            </geometry>
-            <material name="orange"/>
-        </collision>
-        <xacro:inertial_cylinder mass="0.1" length="0.04" radius="0.035">
-            <origin xyz="0 0 0" rpy="0 0 0"/>
-        </xacro:inertial_cylinder>
-    </link>
-    <gazebo reference="right_rear_wheel_link">
-        <material>Gazebo/Orange</material>
-    </gazebo>
-    <!-- RIGHT FRONT WHEEL LINK -->
-    <joint name="right_front_wheel_joint" type="continuous">
-        <parent link="base_link"/>
-        <child link="right_front_wheel_link"/>
-        <origin xyz="0.05 -0.125 0.035" rpy="${pi/2} 0 0"/>
-        <axis xyz="0 0 1"/>
-    </joint>
-    <link name="right_front_wheel_link">
-        <visual>
-            <origin xyz="0 0 0"/>
-            <geometry>
-                <cylinder radius="0.035" length="0.04"/>
-            </geometry>
-            <material name="orange"/>
-        </visual>
-        <collision>
-            <origin xyz="0 0 0"/>
-            <geometry>
-                <cylinder radius="0.035" length="0.04"/>
-            </geometry>
-            <material name="orange"/>
-        </collision>
-        <xacro:inertial_cylinder mass="0.1" length="0.04" radius="0.035">
-            <origin xyz="0 0 0" rpy="0 0 0"/>
-        </xacro:inertial_cylinder>
-    </link>
-    <gazebo reference="right_front_wheel_link">
-        <material>Gazebo/Orange</material>
-        <mu1 value="0.5"/>
-        <mu2 value="0.5"/>
-    </gazebo>
-    <!-- CAMERA STAND LINK -->
-    <joint name="camera_stand_joint" type="fixed">
-        <parent link="base_link"/>
-        <child link="camera_stand_link"/>
-        <origin xyz="0.105 0 0.160" rpy="0 ${pi/2} 0"/>
-    </joint>
-    <link name="camera_stand_link">
-        <visual>
-            <origin xyz="0 0 0"/>
-            <geometry>
-                <box size="0.040 0.040 0.010"/>
-            </geometry>
-            <material name="white"/>
-        </visual>
-        <collision>
-            <origin xyz="0 0 0"/>
-            <geometry>
-                <box size="0.040 0.040 0.010"/>
-            </geometry>
-            <material name="white"/>
-        </collision>
-        <xacro:inertial_box mass="0.100" x="0.040" y="0.040" z="0.010">
-            <origin xyz="0 0 0" rpy="0 0 0"/>
-        </xacro:inertial_box>
-    </link>
-    <gazebo reference="camera_stand_link">
-        <material>Gazebo/White</material>
+    <gazebo reference="right_rear_wheel">
+        <material>Gazebo/Red</material>
     </gazebo>
 </robot>
