Commit message: created urdf and config files for rviz

File: milo_ws/src/milo_description/models/milo_bot/robot.urdf.xacro (robot description, xacro)
@@ -1,5 +1,4 @@
 <?xml version="1.0"?>
 <robot xmlns:xacro="https://www.ros.org/wiki/xacro" name="robot">
-    <!-- <<xacro:include filename="robot_core.xacro" />> -->
-    <link name="base_link"></link>
+    <xacro:include filename="robot_core.xacro" />
 </robot>

Commit message: added diff drive plugin

File: milo_ws/src/milo_description/models/milo_bot/robot.urdf.xacro (robot description, xacro)
@@ -2,4 +2,7 @@
 <robot xmlns:xacro="https://www.ros.org/wiki/xacro" name="robot">
     <xacro:include filename="robot_core.xacro" />
-    <xacro:include filename="gazebo_control.xacro"/>
+    <!-- DIFF DRIVE CONTROL -->
+    <xacro:include filename="diff_drive_control.xacro"/>
+    <!-- SKID STEER CONTROL -->
+    <!-- <xacro:include filename="skid_steer_control.xacro"/> -->
 </robot>

File: milo_ws/src/milo_description/models/milo_bot/robot_core.xacro (robot description, xacro)
@@ -68,6 +68,36 @@
     <gazebo reference="left_rear_wheel">
         <material>Gazebo/Red</material>
+        <!-- <mu2 value="0.3"/>
+        <mu1 value="0.3"/> -->
     </gazebo>
-    <!-- RIGHT WHEEL -->
+    <!-- LEFT FRONT WHEEL -->
+    <joint name="left_front_wheel_joint" type="continuous">
+        <parent link="base_link"/>
+        <child link="left_front_wheel"/>
+        <origin xyz="0.05 0.1125 0" rpy="-${pi/2} 0 0"/>
+        <axis xyz="0 0 1"/>
+    </joint>
+    <link name="left_front_wheel">
+        <visual>
+            <geometry>
+                <cylinder length="0.025" radius="0.035" />
+            </geometry>
+            <material name="blue"/>
+        </visual>
+        <collision>
+            <geometry>
+                <cylinder length="0.025" radius="0.035" />
+            </geometry>
+        </collision>
+        <xacro:inertial_cylinder mass="0.1" length="0.025" radius="0.035">
+            <origin xyz="0 0 0" rpy="0 0 0"/>
+        </xacro:inertial_cylinder>
+    </link>
+    <gazebo reference="left_front_wheel">
+        <material>Gazebo/Red</material>
+        <!-- <mu1 value="0.3"/>
+        <mu2 value="0.3"/> -->
+    </gazebo>
+    <!-- RIGHT REAR WHEEL -->
     <joint name="right_rear_wheel_joint" type="continuous">
         <parent link="base_link"/>
@@ -94,4 +124,34 @@
     <gazebo reference="right_rear_wheel">
         <material>Gazebo/Red</material>
+        <!-- <mu1 value="0.3"/>
+        <mu2 value="0.3"/> -->
+    </gazebo>
+    <!-- RIGHT FRONT WHEEL -->
+    <joint name="right_front_wheel_joint" type="continuous">
+        <parent link="base_link"/>
+        <child link="right_front_wheel"/>
+        <origin xyz="0.050 -0.1125 0" rpy="${pi/2} 0 0"/>
+        <axis xyz="0 0 -1"/>
+    </joint>
+    <link name="right_front_wheel">
+        <visual>
+            <geometry>
+                <cylinder length="0.025" radius="0.035" />
+            </geometry>
+            <material name="blue"/>
+        </visual>
+        <collision>
+            <geometry>
+                <cylinder length="0.025" radius="0.035" />
+            </geometry>
+        </collision>
+        <xacro:inertial_cylinder mass="0.1" length="0.025" radius="0.035">
+            <origin xyz="0 0 0" rpy="0 0 0"/>
+        </xacro:inertial_cylinder>
+    </link>
+    <gazebo reference="right_front_wheel">
+        <material>Gazebo/Red</material>
+        <!-- <mu1 value="0.3"/>
+        <mu2 value="0.3"/> -->
     </gazebo>
 </robot>
