Commit message: added lidar and camera into simulation

File: milo_ws/install/milo_description/share/milo_description/models/milo_bot/robot.urdf.xacro (robot description, xacro)
@@ -6,3 +6,7 @@
     <!-- SKID STEER CONTROL -->
     <xacro:include filename="skid_steer_control.xacro"/>
+    <!-- LiDAR -->
+    <xacro:include filename="lidar.xacro"/>
+    <!-- Camera -->
+    <xacro:include filename="camera.xacro"/>
 </robot>

File: milo_ws/install/milo_description/share/milo_description/models/milo_bot/robot_core.xacro (robot description, xacro)
@@ -14,4 +14,7 @@
         <color rgba="0 0 0 1"/>
     </material>
+    <material name="red">
+        <color rgba="1 0 0 1"/>
+    </material>
     <link name="base_link">
     </link>
@@ -28,5 +31,5 @@
                 <box size="0.220 0.210 0.105"/>
             </geometry>
-            <material name="white"/>
+            <material name="blue"/>
         </visual>
         <collision>
@@ -41,5 +44,5 @@
     </link>
     <gazebo reference="chassis">
-        <material>Gazebo/White</material>
+        <material>Gazebo/Blue</material>
     </gazebo>
     <!-- LEFT REAR WHEEL -->
@@ -55,5 +58,5 @@
                 <cylinder length="0.025" radius="0.035" />
             </geometry>
-            <material name="blue"/>
+            <material name="red"/>
         </visual>
         <collision>
@@ -61,5 +64,5 @@
                 <cylinder length="0.025" radius="0.035" />
             </geometry>
-            <material name="blue"/>
+            <material name="red"/>
         </collision>
         <xacro:inertial_cylinder mass="0.1" length="0.025" radius="0.035">
@@ -84,5 +87,5 @@
                 <cylinder length="0.025" radius="0.035" />
             </geometry>
-            <material name="blue"/>
+            <material name="red"/>
         </visual>
         <collision>
@@ -90,5 +93,5 @@
                 <cylinder length="0.025" radius="0.035" />
             </geometry>
-            <material name="blue"/>
+            <material name="red"/>
         </collision>
         <xacro:inertial_cylinder mass="0.1" length="0.025" radius="0.035">
@@ -113,5 +116,5 @@
                 <cylinder length="0.025" radius="0.035" />
             </geometry>
-            <material name="blue"/>
+            <material name="red"/>
         </visual>
         <collision>
@@ -119,5 +122,5 @@
                 <cylinder length="0.025" radius="0.035" />
             </geometry>
-            <material name="blue"/>
+            <material name="red"/>
         </collision>
         <xacro:inertial_cylinder mass="0.1" length="0.025" radius="0.035">
@@ -142,5 +145,5 @@
                 <cylinder length="0.025" radius="0.035" />
             </geometry>
-            <material name="blue"/>
+            <material name="red"/>
         </visual>
         <collision>
@@ -148,5 +151,5 @@
                 <cylinder length="0.025" radius="0.035" />
             </geometry>
-            <material name="blue"/>
+            <material name="red"/>
         </collision>
         <xacro:inertial_cylinder mass="0.1" length="0.025" radius="0.035">
