Commit message: added ros2 diff_drive controller

File: milo_ws/install/milo_description/share/milo_description/models/milo_bot/lidar.xacro (robot description, xacro)
@@ -44,5 +44,5 @@
             <plugin name="laser_controller" filename="libgazebo_ros_ray_sensor.so">
                 <ros>
-                    <argument>~/out:=scan</argument>
+                    <remapping>~/out:=scan</remapping>
                 </ros>
                 <output_type>sensor_msgs/LaserScan</output_type>

File: milo_ws/install/milo_description/share/milo_description/models/milo_bot/robot.urdf.xacro (robot description, xacro)
@@ -1,9 +1,18 @@
 <?xml version="1.0"?>
 <robot xmlns:xacro="https://www.ros.org/wiki/xacro" name="robot">
+    <xacro:arg name="use_ros2_control" default="true" />
+    <xacro:if value="$(arg use_ros2_control)">
+        <xacro:include filename="ros2_control.xacro"/>
+    </xacro:if>
+    <xacro:unless value="$(arg use_ros2_control)">
+        <xacro:include filename="skid_steer_control.xacro"/>
+    </xacro:unless>
     <xacro:include filename="robot_core.xacro" />
     <!-- DIFF DRIVE CONTROL -->
     <!-- <xacro:include filename="diff_drive_control.xacro"/> -->
     <!-- SKID STEER CONTROL -->
-    <xacro:include filename="skid_steer_control.xacro"/>
+    <!-- <xacro:include filename="skid_steer_control.xacro"/> -->
+    <!-- CUSTOM ROS2 CONTROL -->
+    <!-- <xacro:include filename="ros2_control.xacro" /> -->
     <!-- LiDAR -->
     <xacro:include filename="lidar.xacro"/>

File: milo_ws/install/milo_description/share/milo_description/models/milo_bot/robot_core.xacro (robot description, xacro)
@@ -19,4 +19,11 @@
     <link name="base_link">
     </link>
+  <!-- ROBOT FOOTPRINT -->
+  <link name="base_footprint"/>
+  <joint name="base_joint" type="fixed">
+    <parent link="base_link"/>
+    <child link="base_footprint"/>
+    <origin xyz="0.0 0.0 -0.035" rpy="0 0 0"/>
+  </joint>
     <!-- CHASSIS -->
     <joint name="chassis_joint" type="fixed">
@@ -48,7 +55,7 @@
     <!-- LEFT REAR WHEEL -->
     <joint name="left_rear_wheel_joint" type="continuous">
-        <parent link="base_link"/>
+        <parent link="chassis"/>
         <child link="left_rear_wheel"/>
-        <origin xyz="-0.05 0.1175 0" rpy="-${pi/2} 0 0"/>
+        <origin xyz="-0.05 0.1175 -0.0525" rpy="-${pi/2} 0 0"/>
         <axis xyz="0 0 1"/>
     </joint>
@@ -62,11 +69,11 @@
         <collision>
             <geometry>
-                <cylinder length="0.025" radius="0.035" />
+                <sphere radius="0.035" />
             </geometry>
             <material name="red"/>
         </collision>
-        <xacro:inertial_cylinder mass="0.1" length="0.025" radius="0.035">
+        <xacro:inertial_sphere mass="0.1" radius="0.035">
             <origin xyz="0 0 0" rpy="0 0 0"/>
-        </xacro:inertial_cylinder>
+        </xacro:inertial_sphere>
     </link>
     <gazebo reference="left_rear_wheel">
@@ -77,7 +84,7 @@
     <!-- LEFT FRONT WHEEL -->
     <joint name="left_front_wheel_joint" type="continuous">
-        <parent link="base_link"/>
+        <parent link="chassis"/>
         <child link="left_front_wheel"/>
-        <origin xyz="0.05 0.1175 0" rpy="-${pi/2} 0 0"/>
+        <origin xyz="0.05 0.1175 -0.0525" rpy="-${pi/2} 0 0"/>
         <axis xyz="0 0 1"/>
     </joint>
@@ -91,11 +98,11 @@
         <collision>
             <geometry>
-                <cylinder length="0.025" radius="0.035" />
+                <sphere radius="0.035" />
             </geometry>
             <material name="red"/>
         </collision>
-        <xacro:inertial_cylinder mass="0.1" length="0.025" radius="0.035">
+        <xacro:inertial_sphere mass="0.1" radius="0.035">
             <origin xyz="0 0 0" rpy="0 0 0"/>
-        </xacro:inertial_cylinder>
+        </xacro:inertial_sphere>
     </link>
     <gazebo reference="left_front_wheel">
@@ -106,7 +113,7 @@
     <!-- RIGHT REAR WHEEL -->
     <joint name="right_rear_wheel_joint" type="continuous">
-        <parent link="base_link"/>
+        <parent link="chassis"/>
         <child link="right_rear_wheel"/>
-        <origin xyz="-0.05 -0.1175 0" rpy="${pi/2} 0 0"/>
+        <origin xyz="-0.05 -0.1175 -0.0525" rpy="${pi/2} 0 0"/>
         <axis xyz="0 0 -1"/>
     </joint>
@@ -120,11 +127,11 @@
         <collision>
             <geometry>
-                <cylinder length="0.025" radius="0.035" />
+                <sphere radius="0.035" />
             </geometry>
             <material name="red"/>
         </collision>
-        <xacro:inertial_cylinder mass="0.1" length="0.025" radius="0.035">
+        <xacro:inertial_sphere mass="0.1" radius="0.035">
             <origin xyz="0 0 0" rpy="0 0 0"/>
-        </xacro:inertial_cylinder>
+        </xacro:inertial_sphere>
     </link>
     <gazebo reference="right_rear_wheel">
@@ -135,7 +142,7 @@
     <!-- RIGHT FRONT WHEEL -->
     <joint name="right_front_wheel_joint" type="continuous">
-        <parent link="base_link"/>
+        <parent link="chassis"/>
         <child link="right_front_wheel"/>
-        <origin xyz="0.05 -0.1175 0" rpy="${pi/2} 0 0"/>
+        <origin xyz="0.05 -0.1175 -0.0525" rpy="${pi/2} 0 0"/>
         <axis xyz="0 0 -1"/>
     </joint>
@@ -149,11 +156,11 @@
         <collision>
             <geometry>
-                <cylinder length="0.025" radius="0.035" />
+                <sphere radius="0.035" />
             </geometry>
             <material name="red"/>
         </collision>
-        <xacro:inertial_cylinder mass="0.1" length="0.025" radius="0.035">
+        <xacro:inertial_sphere mass="0.1" radius="0.035">
             <origin xyz="0 0 0" rpy="0 0 0"/>
-        </xacro:inertial_cylinder>
+        </xacro:inertial_sphere>
     </link>
     <gazebo reference="right_front_wheel">

Commit message: fixed up simulation - world file, launch files, lidar visualisation

File: milo_ws/install/milo_description/share/milo_description/models/milo_bot/lidar.xacro (robot description, xacro)
@@ -27,5 +27,5 @@
         <sensor name="laser" type="ray">
             <pose> 0 0 0 0 0 0 </pose>
-            <visualize>false</visualize>
+            <visualize>true</visualize>
             <update_rate>5.5</update_rate>
             <ray>
@@ -44,5 +44,5 @@
             <plugin name="laser_controller" filename="libgazebo_ros_ray_sensor.so">
                 <ros>
-                    <remapping>~/out:=scan</remapping>
+                    <remap>~/out:=scan</remap>
                 </ros>
                 <output_type>sensor_msgs/LaserScan</output_type>

File: milo_ws/install/milo_description/share/milo_description/models/milo_bot/robot_core.xacro (robot description, xacro)
@@ -55,7 +55,7 @@
     <!-- LEFT REAR WHEEL -->
     <joint name="left_rear_wheel_joint" type="continuous">
-        <parent link="chassis"/>
+        <parent link="base_link"/>
         <child link="left_rear_wheel"/>
-        <origin xyz="-0.05 0.1175 -0.0525" rpy="-${pi/2} 0 0"/>
+        <origin xyz="-0.05 0.1175 0.0" rpy="-${pi/2} 0 0"/>
         <axis xyz="0 0 1"/>
     </joint>
@@ -84,7 +84,7 @@
     <!-- LEFT FRONT WHEEL -->
     <joint name="left_front_wheel_joint" type="continuous">
-        <parent link="chassis"/>
+        <parent link="base_link"/>
         <child link="left_front_wheel"/>
-        <origin xyz="0.05 0.1175 -0.0525" rpy="-${pi/2} 0 0"/>
+        <origin xyz="0.05 0.1175 0.0" rpy="-${pi/2} 0 0"/>
         <axis xyz="0 0 1"/>
     </joint>
@@ -113,7 +113,7 @@
     <!-- RIGHT REAR WHEEL -->
     <joint name="right_rear_wheel_joint" type="continuous">
-        <parent link="chassis"/>
+        <parent link="base_link"/>
         <child link="right_rear_wheel"/>
-        <origin xyz="-0.05 -0.1175 -0.0525" rpy="${pi/2} 0 0"/>
+        <origin xyz="-0.05 -0.1175 0.0" rpy="${pi/2} 0 0"/>
         <axis xyz="0 0 -1"/>
     </joint>
@@ -142,7 +142,7 @@
     <!-- RIGHT FRONT WHEEL -->
     <joint name="right_front_wheel_joint" type="continuous">
-        <parent link="chassis"/>
+        <parent link="base_link"/>
         <child link="right_front_wheel"/>
-        <origin xyz="0.05 -0.1175 -0.0525" rpy="${pi/2} 0 0"/>
+        <origin xyz="0.05 -0.1175 0.0" rpy="${pi/2} 0 0"/>
         <axis xyz="0 0 -1"/>
     </joint>
