Commit message: feature/milo-slam: Added ekf localisation for encoder plugin and imu plugin

File: milo_ws/src/simulation/milo_description/models/milo_bot/controllers/diff_drive_control.xacro (robot description, xacro)
@@ -6,7 +6,7 @@
 <!-- Controller for 4-wheeled robot (skid_steer_drive) -->
 <gazebo>
-<plugin name='skid_steer_drive' filename='libgazebo_ros_diff_drive.so'>
+<plugin name='diff_drive' filename='libgazebo_ros_diff_drive.so'>
     <ros>
-        <namespace> </namespace>
+        <namespace>diff_drive</namespace>
     </ros>
     <num_wheel_pairs>2</num_wheel_pairs>
@@ -16,6 +16,6 @@
     <right_joint>right_front_wheel_joint</right_joint>
     <!-- Kinematics -->
-    <wheel_separation>0.180</wheel_separation>
-    <wheel_separation>0.180</wheel_separation>
+    <wheel_separation>0.235</wheel_separation>
+    <wheel_separation>0.235</wheel_separation>
     <wheel_diameter>0.070</wheel_diameter>
     <wheel_diameter>0.070</wheel_diameter>
@@ -25,5 +25,5 @@
     <!-- Output -->
     <publish_odom>true</publish_odom>
-    <publish_odom_tf>true</publish_odom_tf>
+    <publish_odom_tf>false</publish_odom_tf>
     <publish_wheel_tf>true</publish_wheel_tf>
     <odometry_frame>odom</odometry_frame>

File: milo_ws/src/simulation/milo_description/models/milo_bot/lidars/lidar.xacro (robot description, xacro)
@@ -44,5 +44,6 @@
             <plugin name="laser_controller" filename="libgazebo_ros_ray_sensor.so">
                 <ros>
-                    <remap>~/out:=scan</remap>
+                    <namespace>/milo</namespace>
+                    <remapping>~/out:=scan</remapping>
                 </ros>
                 <output_type>sensor_msgs/LaserScan</output_type>

File: milo_ws/src/simulation/milo_description/models/milo_bot/robot.urdf.xacro (robot description, xacro)
@@ -3,12 +3,12 @@
     <xacro:include filename="robot_core.xacro" />
     <!-- DIFF DRIVE CONTROL -->
-    <!-- <xacro:include filename="diff_drive_control.xacro"/> -->
-    <!-- SKID STEER CONTROL -->
-    <!-- <xacro:include filename="skid_steer_control.xacro"/> -->
-    <!-- CUSTOM ROS2 CONTROL -->
-    <xacro:include filename="ros2_control.xacro" />
+    <xacro:include filename="controllers/diff_drive_control.xacro"/>
+    <!-- CUSTOM ROS2 CONTROL - currently laser scanner moves in rviz bug-->
+    <!-- <xacro:include filename="ros2_control.xacro" /> -->
     <!-- LiDAR -->
-    <xacro:include filename="lidar.xacro"/>
+    <xacro:include filename="lidars/lidar.xacro"/>
     <!-- Camera -->
-    <xacro:include filename="camera.xacro"/>
+    <xacro:include filename="cameras/camera.xacro"/>
+    <!-- IMU -->
+    <xacro:include filename="imu/imu.xacro"/>
 </robot>

File: milo_ws/src/simulation/milo_description/models/milo_bot/robot_core.xacro (robot description, xacro)
@@ -16,4 +16,7 @@
     <material name="red">
         <color rgba="1 0 0 1"/>
+    </material>
+    <material name="purple">
+        <color rgba="0.5 0.0 0.5 1.0"/>
     </material>
     <link name="base_link">
@@ -79,6 +82,6 @@
     <gazebo reference="left_rear_wheel">
         <material>Gazebo/Red</material>
+        <mu2 value="0.2"/>
         <mu1 value="0.2"/>
-        <mu2 value="0.2"/>
     </gazebo>
     <!-- LEFT FRONT WHEEL -->
