Commit message: PDR-2 Set up rtabslam

File: milo_ws/src/milo_description/models/milo_bot/controllers/ros2_control.xacro (robot description, xacro)
@@ -41,5 +41,5 @@
     <gazebo>
         <plugin filename="libgazebo_ros2_control.so" name="gazebo_ros2_control">
-            <parameters>$(find milo_description)/config/my_controllers.yaml</parameters>
+            <parameters>$(find milo_description)/config/my_controllers.yml</parameters>
         </plugin>
     </gazebo>

File: milo_ws/src/milo_description/models/milo_bot/robot_core.xacro (robot description, xacro)
@@ -16,4 +16,7 @@
     <material name="red">
         <color rgba="1 0 0 1"/>
+    </material>
+    <material name="purple">
+        <color rgba="0.5 0 0.5 1"/>
     </material>
     <link name="base_link">

File: milo_ws/src/milo_description/models/milo_bot/sensors/camera.xacro (robot description, xacro)
@@ -27,9 +27,9 @@
             <update_rate>10</update_rate>
             <camera>
-                <horizontal_fov>2.094</horizontal_fov>
+                <horizontal_fov>1.309</horizontal_fov>
                 <image>
                     <format>R8G8B8</format>
-                    <width>4608</width>
-                    <height>2592</height>
+                    <width>4056</width>
+                    <height>3040</height>
                 </image>
                 <clip>
@@ -40,4 +40,16 @@
             <plugin name="camera_controller" filename="libgazebo_ros_camera.so">
                 <frame_name>camera_link_optical</frame_name>
+                <!-- <alwaysOn>true</alwaysOn>
+                <updateRate>0.0</updateRate>
+                <cameraName>rrbot/camera1</cameraName>
+                <imageTopicName>image_raw</imageTopicName>
+                <cameraInfoTopicName>camera_info</cameraInfoTopicName>
+                <frameName>camera_link</frameName>
+                <hackBaseline>0.07</hackBaseline>
+                <distortionK1>0.0</distortionK1>
+                <distortionK2>0.0</distortionK2>
+                <distortionK3>0.0</distortionK3>
+                <distortionT1>0.0</distortionT1>
+                <distortionT2>0.0</distortionT2> -->
             </plugin>
         </sensor>
